Commit message: Add script to regenerate urdf using onshape-to-robot

File: src/robot_description/urdf/robot.urdf (robot description, URDF)
Before this commit: robot robot, 6 links, 5 joints
Links:
- added link end_effector, mass 1e-9
Joints:
- added joint end_effector_frame: type fixed, parent part_14, child end_effector, origin xyz=0.0115 0.123706 0.004 rpy=1.5708 -2.81638e-15 3.14159, axis 0 0 0
- joint joint_1: limit lower=-0.678448 upper=2.46314 effort=10 velocity=10 -> lower=0 upper=3.14159 effort=10 velocity=20.5; origin xyz=-2.08489e-08 1.03674e-08 0.056 rpy=-3.14159 1.84871e-18 -2.24924 -> xyz=-2.08489e-08 1.03674e-08 0.056 rpy=-3.14159 -5.54668e-32 -1.5708
- joint joint_2: limit lower=-0.134493 upper=3.0071 effort=10 velocity=10 -> lower=0 upper=3.14159 effort=10 velocity=20.5; origin xyz=-0.004 -0.0139185 -0.0402765 rpy=1.5708 1.4363 1.5708 -> xyz=-0.004 -0.0139185 -0.0402765 rpy=-3.33067e-16 1.5708 0
- joint joint_3: limit lower=-2.17609 upper=0.965502 effort=10 velocity=10 -> lower=0 upper=3.14159 effort=10 velocity=20.5; origin xyz=-4.04768e-09 -0.12 8.58688e-17 rpy=2.50215e-15 5.38531e-15 0.605294 -> xyz=-4.04768e-09 -0.12 -1.47451e-17 rpy=-9.99201e-16 9.99201e-16 -1.5708
- joint joint_4: limit lower=-0.0418501 upper=3.09974 effort=10 velocity=10 -> lower=0 upper=3.14159 effort=10 velocity=20.5; origin xyz=-0.0053 -0.08975 -0.0075 rpy=-1.5708 -1.52895 -7.62844e-14 -> xyz=-0.0053 -0.08975 -0.0075 rpy=-1.5708 -1.5708 0
- joint joint_5: limit lower=-1.15837 upper=1.98322 effort=10 velocity=10 -> lower=0 upper=3.14159 effort=10 velocity=20.5; origin xyz=0.005 -0.014 -0.028 rpy=-1.5708 -0.412425 -7.74018e-15 -> xyz=0.005 -0.014 -0.028 rpy=-1.5708 -1.5708 0
